File: PCB/IMU controller.kicad_pcb (KiCad board)
At the start: 4 copper layers, 30 x 30 mm, 38 parts, among them J1 Conn_01x05, U1 NRF52810-QFAA-R, U2 FC31M2-32.768-N09LLDT, U3 BMI270, U6 PTS526SMG15SMTR21 LFS, X1 S3232000081040

Commit message: added updated PCB files
Parts:
- removed C15, C16: 10uF, Capacitor_SMD:C_0805_2012Metric
- removed C17: 1uF, Capacitor_SMD:C_0603_1608Metric
- removed C18: 100nF, Capacitor_SMD:C_0402_1005Metric
- removed L1: 2.2uH, Inductor_SMD:L_0805_2012Metric
- removed LED1: SZYY1615RGB-B 4PIN, EasyEDA:LED-SMD_4P-L1.6-W1.5-TR-1
- removed R2: 1.6k-2.4k, Resistor_SMD:R_0603_1608Metric
- removed R3: 390-430, Resistor_SMD:R_0603_1608Metric
- removed R4: 23.7k, Resistor_SMD:R_0603_1608Metric
- removed Uu4: MAX17223ELT+T, EasyEDA:UDFN-6_L2.0-W2.0-P0.65-BL
- added U4: LS L29K-G1J2-1-Z, EasyEDA:LED-SMD_L1.3-W0.8-LS1.7-FD, B.Cu at (141.5, 82.2)
- R1: value 910-1k -> 620
- moved C14 21.1 mm to (144.7, 77.0), turned to 180 degrees
- moved R1 3.50 mm to (145.2, 83.0), turned to 180 degrees
Connections:
- R1 pad 1: RED -> VDD
- U1 pad 16: EN -> LED
- U1 pad 17: RED -> unconnected-(U1-P0.14-Pad17)
- U1 pad 18: GREEN -> unconnected-(U1-P0.15-Pad18)
- U1 pad 19: BLUE -> unconnected-(U1-P0.16-Pad19)
Routing:
- net 4V: track 13.2 -> 0.00 mm
- net EN: track 11.0 -> 0.00 mm, vias 2 -> 0
- net VDD: track 66.5 -> 59.0 mm
- net GND: track 68.8 -> 62.7 mm, vias 60 -> 56
- net LX: track 3.96 -> 0.00 mm
- net Net-(Uu4-SEL): track 3.85 -> 0.00 mm
- net LED: track 0.00 -> 3.37 mm
- net RED: track 3.05 -> 0.00 mm
- net GREEN: track 2.55 -> 0.00 mm
- net BLUE: track 2.38 -> 0.00 mm
- net Net-(LED1-G): track 2.00 -> 0.00 mm
- net Net-(LED1-B): track 1.94 -> 0.00 mm
- net Net-(U4-A): track 3.64 -> 2.87 mm
